Commit message: Added fixed xacros. Robot generation working

File: lab2/robot/links_and_joints.urdf.xacro (robot description, xacro)
@@ -1,8 +1,9 @@
 <robot name="robot" xmlns:xacro="http://www.ros.org/wiki/xacro">
-  <xacro:include filename="$(find lab2)/robot/materials.xacro.xml" />
+  <xacro:include filename="$(find lab2)/materials.urdf.xacro" />
     <xacro:macro name="m_link_cylinder" params="name origin_xyz origin_rpy radius length material">
         <link name="${name}">
           <inertial>
-            <origin rpy="${origin_rpy}" xyz="${origin_xyz}" />
+            <mass value="10" />
+            <inertia ixx="100" ixy="0" ixz="0" iyy="100" iyz="0" izz="100" />
           </inertial>
           <collision>
@@ -34,5 +35,4 @@
       <inertial>
         <mass value="10" />
-        <origin rpy="${origin_rpy}" xyz="${origin_xyz}" />
         <inertia ixx="100" ixy="0" ixz="0" iyy="100" iyz="0" izz="100" />
       </inertial>

File: lab2/robot/load_params.urdf.xacro (robot description, xacro)
@@ -1,5 +1,5 @@
 <?xml version="1.0" ?>
 <robot name="robot" xmlns:xacro="http://www.ros.org/wiki/xacro">
-  <xacro:property name="yaml_file" value="$(find lab2)/config/params.yaml" />
+  <xacro:property name="yaml_file" value="$(find lab2)/params.yaml" />
   <xacro:property name="params" value="${load_yaml(yaml_file)}"/>
   <xacro:property name="a1" value="${params['a1']}" />

File: lab2/robot/materials.urdf.xacro (robot description, xacro)
@@ -1,4 +1,4 @@
 <?xml version="1.0"?>
-<robot name="$(arg robot_name)" xmlns:xacro="http://www.ros.org/wiki/xacro">
+<robot name="robot" xmlns:xacro="http://www.ros.org/wiki/xacro">
 <material name="black">
   <color rgba="0.0 0.0 0.0 1.0"/>

File: lab2/robot/robot.urdf.xacro (robot description, xacro)
@@ -1,6 +1,6 @@
 <robot name="robot" xmlns:xacro="http://www.ros.org/wiki/xacro">
   <!-- BGN - Include -->
-  <xacro:include filename="$(find lab2)/robot/load_params.xacro.xml" />
-  <xacro:include filename="$(find lab2)/robot/links_and_joints.xacro.xml" />
+  <xacro:include filename="$(find lab2)/load_params.urdf.xacro" />
+  <xacro:include filename="$(find lab2)/links_and_joints.urdf.xacro" />
   <!-- END - Include -->
   <!-- BGN - Robot description -->
@@ -15,11 +15,11 @@
     axis_xyz="0 0 1"
     origin_rpy="0 0 0"
-    origin_xyz="0 0 0"
+    origin_xyz="0 0 0.05"
     parent="base"
     child="base_ext"
-    limit_l="-3.14" limit_u="3.14">
+    limit_lower="0" limit_upper="0">
   </xacro:m_joint>
   <xacro:m_link_cylinder name="base_ext"
-    origin_xyz="${a1/2} 0 {d1/2}"
+    origin_xyz="${a1/2} 0 ${d1/2}"
     origin_rpy="0 0 0"
     radius="0.05"
@@ -30,13 +30,13 @@
     type="revolute"
     axis_xyz="0 0 1"
-    origin_rpy="-1.57 0 0"
+    origin_rpy="0 0 0"
     origin_xyz="0 0 0"
     parent="base_ext"
     child="arm"
-    limit_l="-3.14" limit_u="3.14">
+    limit_lower="0" limit_upper="0">
   </xacro:m_joint>
   <xacro:m_link_cylinder name="arm"
-    origin_xyz="${a2/2} 0 {d2/2}"
-    origin_rpy="${pi/2} 0 0"
+    origin_xyz="${a2/2} 0 ${d2/2}"
+    origin_rpy="0 ${pi/2} 0"
     radius="0.05"
     length="${a2}"
@@ -46,13 +46,13 @@
     type="revolute"
     axis_xyz="0 0 1"
-    origin_rpy="0 0 0"
-    origin_xyz="0 0 0"
+    origin_rpy="${-pi/2} 0 0"
+    origin_xyz="${a2} 0 0"
     parent="arm"
     child="hand"
-    limit_l="-3.14" limit_u="3.14">
+    limit_lower="-3.14" limit_upper="3.14">
   </xacro:m_joint>
   <xacro:m_link_cylinder name="hand"
-    origin_xyz="${a3/2} 0 {d3/2}"
-    origin_rpy="0 0 0"
+    origin_xyz="${a3/2} 0 ${d3/2}"
+    origin_rpy="0 ${pi/2} 0"
     radius="0.05"
     length="${a3}"

Commit message: Added tool

File: lab2/robot/links_and_joints.urdf.xacro (robot description, xacro)
@@ -52,3 +52,19 @@
     </link>
   </xacro:macro>
+  <xacro:macro name="m_gun" params="name origin_xyz origin_rpy scale">
+    <link name="${name}">
+      <!-- <collision>
+        <origin rpy="${origin_rpy}" xyz="${origin_xyz}" />
+        <geometry>
+          <box size="${size}" />
+        </geometry>
+      </collision> -->
+      <visual>
+        <origin rpy="${origin_rpy}" xyz="${origin_xyz}" />
+        <geometry>
+          <mesh filename = "package://lab2/gatling.stl" scale="${scale}"/>
+        </geometry>
+      </visual>
+    </link>
+  </xacro:macro>
 </robot>

File: lab2/robot/robot.urdf.xacro (robot description, xacro)
@@ -59,4 +59,18 @@
     material="white">
   </xacro:m_link_cylinder>
+  <xacro:m_joint name="hand-tool"
+  type="revolute"
+  axis_xyz="0 0 1"
+  origin_rpy="0 0 0"
+  origin_xyz="${a3} 0 ${d3}"
+  parent="hand"
+  child="tool"
+  limit_lower="0" limit_upper="0">
+  </xacro:m_joint>
+  <xacro:m_gun name="tool"
+    origin_xyz="0 0 0"
+    origin_rpy="0 0 0"
+    scale="0.001 0.001 0.001">
+  </xacro:m_gun>
   <!-- END - Robot description -->
 </robot>
