Commit message: Added working non_kdl. not great not terrible

File: lab3/robot/links_and_joints.urdf.xacro (robot description, xacro)
@@ -68,3 +68,19 @@
     </link>
   </xacro:macro>
+  <xacro:macro name="m_tool" params="name origin_xyz origin_rpy">
+    <link name="${name}">
+      <!-- <collision>
+        <origin rpy="${origin_rpy}" xyz="${origin_xyz}" />
+        <geometry>
+          <box size="${size}" />
+        </geometry>
+      </collision> -->
+      <visual>
+        <origin rpy="${origin_rpy}" xyz="${origin_xyz}" />
+        <geometry>
+          <cylinder radius="0.01" length="0.05" />
+        </geometry>
+      </visual>
+    </link>
+  </xacro:macro>
 </robot>

File: lab3/robot/robot.urdf.xacro (robot description, xacro)
@@ -60,5 +60,5 @@
   </xacro:m_link_cylinder>
   <xacro:m_joint name="hand-tool"
-  type="revolute"
+  type="fixed"
   axis_xyz="0 0 1"
   origin_rpy="0 0 0"
@@ -68,9 +68,14 @@
   limit_lower="0" limit_upper="0">
   </xacro:m_joint>
-  <xacro:m_gun name="tool"
+  <xacro:m_tool name="tool"
+    origin_xyz="0 0 0"
+    origin_rpy="0 0 0">
+  </xacro:m_tool>
+  <!-- <xacro:m_gun name="tool"
     origin_xyz="0 0 0"
     origin_rpy="0 0 0"
     scale="0.001 0.001 0.001">
   </xacro:m_gun>
+ -->
   <!-- END - Robot description -->
 </robot>

Commit message: Refaktoryzacja kodu

File: lab3/robot/links_and_joints.urdf.xacro (robot description, xacro)
@@ -68,3 +68,19 @@
     </link>
   </xacro:macro>
+  <xacro:macro name="m_tool" params="name origin_xyz origin_rpy">
+    <link name="${name}">
+      <!-- <collision>
+        <origin rpy="${origin_rpy}" xyz="${origin_xyz}" />
+        <geometry>
+          <box size="${size}" />
+        </geometry>
+      </collision> -->
+      <visual>
+        <origin rpy="${origin_rpy}" xyz="${origin_xyz}" />
+        <geometry>
+          <cylinder radius="0.01" length="0.05" />
+        </geometry>
+      </visual>
+    </link>
+  </xacro:macro>
 </robot>

File: lab3/robot/load_params.urdf.xacro (robot description, xacro)
@@ -3,10 +3,12 @@
   <xacro:property name="yaml_file" value="$(find lab3)/params.yaml" />
   <xacro:property name="params" value="${load_yaml(yaml_file)}"/>
-  <xacro:property name="a1" value="${params['a1']}" />
-  <xacro:property name="d1" value="${ params['d1']}" />
-  <xacro:property name="a2" value="${params['a2']}" />
-  <xacro:property name="d2" value="${params['d2']}" />
-  <xacro:property name="a3" value="${params['a3']}" />
-  <xacro:property name="d3" value="${params['d3']}" />
+  <xacro:property name="a0" value="${params['base']['a']}" />
+  <xacro:property name="d0" value="${params['base']['d']}" />
+  <xacro:property name="a1" value="${params['base_ext']['a']}" />
+  <xacro:property name="d1" value="${params['base_ext']['d']}" />
+  <xacro:property name="a2" value="${params['arm']['a']}" />
+  <xacro:property name="d2" value="${params['arm']['d']}" />
+  <xacro:property name="a3" value="${params['hand']['a']}" />
+  <xacro:property name="d3" value="${params['hand']['d']}" />
   <xacro:property name="link_00_name" value="base" />
   <xacro:property name="link_01_name" value="base_ext" />

File: lab3/robot/robot.urdf.xacro (robot description, xacro)
@@ -15,5 +15,5 @@
     axis_xyz="0 0 1"
     origin_rpy="0 0 0"
-    origin_xyz="0 0 0.05"
+    origin_xyz="0 0 ${d0}"
     parent="base"
     child="base_ext"
@@ -60,5 +60,5 @@
   </xacro:m_link_cylinder>
   <xacro:m_joint name="hand-tool"
-  type="revolute"
+  type="fixed"
   axis_xyz="0 0 1"
   origin_rpy="0 0 0"
@@ -68,9 +68,14 @@
   limit_lower="0" limit_upper="0">
   </xacro:m_joint>
-  <xacro:m_gun name="tool"
+  <xacro:m_tool name="tool"
+    origin_xyz="0 0 0"
+    origin_rpy="0 0 0">
+  </xacro:m_tool>
+  <!-- <xacro:m_gun name="tool"
     origin_xyz="0 0 0"
     origin_rpy="0 0 0"
     scale="0.001 0.001 0.001">
   </xacro:m_gun>
+ -->
   <!-- END - Robot description -->
 </robot>

Commit message: Dodano narzędzie

File: lab3/robot/links_and_joints.urdf.xacro (robot description, xacro)
@@ -79,6 +79,7 @@
         <origin rpy="${origin_rpy}" xyz="${origin_xyz}" />
         <geometry>
-          <cylinder radius="0.01" length="0.05" />
+          <cylinder radius="0.02" length="0.2" />
         </geometry>
+        <material name="orange" />
       </visual>
     </link>

File: lab3/robot/robot.urdf.xacro (robot description, xacro)
@@ -68,10 +68,7 @@
   limit_lower="0" limit_upper="0">
   </xacro:m_joint>
-<<<<<<< HEAD
-=======
->>>>>>> refaktoryzacja
   <xacro:m_tool name="tool"
     origin_xyz="0 0 0"
-    origin_rpy="0 0 0">
+    origin_rpy="0 -1.57 0">
   </xacro:m_tool>
   <!-- <xacro:m_gun name="tool"

Commit message: Dodano strzałki, dodanie pliku konfiguracyjnego robot/robot_ready.rviz z gotowymi ustawieniami do demonstracji, dodanie ilustracji do dokumentacji

File: lab3/robot/links_and_joints.urdf.xacro (robot description, xacro)
@@ -79,5 +79,5 @@
         <origin rpy="${origin_rpy}" xyz="${origin_xyz}" />
         <geometry>
-          <cylinder radius="0.02" length="0.2" />
+          <cylinder radius="0.051" length="0.005" />
         </geometry>
         <material name="orange" />
