Commit message: Wstępna wersja, robot się rusza

File: lab5/robot/links_and_joints.urdf.xacro (robot description, xacro)
@@ -1,4 +1,4 @@
 <robot name="robot" xmlns:xacro="http://www.ros.org/wiki/xacro">
-  <xacro:include filename="$(find lab3)/materials.urdf.xacro" />
+  <xacro:include filename="$(find lab5)/materials.urdf.xacro" />
     <xacro:macro name="m_link_cylinder" params="name origin_xyz origin_rpy radius length material">
         <link name="${name}">
@@ -63,5 +63,5 @@
         <origin rpy="${origin_rpy}" xyz="${origin_xyz}" />
         <geometry>
-          <mesh filename = "package://lab3/gatling.stl" scale="${scale}"/>
+          <mesh filename = "package://lab5/gatling.stl" scale="${scale}"/>
         </geometry>
       </visual>

File: lab5/robot/load_params.urdf.xacro (robot description, xacro)
@@ -1,5 +1,5 @@
 <?xml version="1.0" ?>
 <robot name="robot" xmlns:xacro="http://www.ros.org/wiki/xacro">
-  <xacro:property name="yaml_file" value="$(find lab3)/params.yaml" />
+  <xacro:property name="yaml_file" value="$(find lab5)/params.yaml" />
   <xacro:property name="params" value="${load_yaml(yaml_file)}"/>
   <xacro:property name="a0" value="${params['base']['a']}" />

File: lab5/robot/robot.urdf.xacro (robot description, xacro)
@@ -1,6 +1,6 @@
 <robot name="robot" xmlns:xacro="http://www.ros.org/wiki/xacro">
   <!-- BGN - Include -->
-  <xacro:include filename="$(find lab3)/load_params.urdf.xacro" />
-  <xacro:include filename="$(find lab3)/links_and_joints.urdf.xacro" />
+  <xacro:include filename="$(find lab5)/load_params.urdf.xacro" />
+  <xacro:include filename="$(find lab5)/links_and_joints.urdf.xacro" />
   <!-- END - Include -->
   <!-- BGN - Robot description -->
